File: USBC.kicad_sch (KiCad schematic)
At the start: 4 parts, among them J1 USB_C_Receptacle

Commit message: Updated PCB
Parts:
- F1: value 0.35A -> 0.75A
Changed lines of the file:
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@@
 			)
 		)
-		(property "Value" "0.35A"
+		(property "Value" "0.75A"
 			(at 157.48 63.5 90)
 			(show_name no)
