File: ocp.kicad_sch (KiCad schematic)
At the start: 13 parts, among them J1 ADS1115, J2 Screw_Terminal_01x03, J3 Screw_Terminal_01x02, U2 REF3033, U3 TL072

Commit message: v2
Parts:
- removed J2: Screw_Terminal_01x03, TerminalBlock_Phoenix:TerminalBlock_Phoenix_MKDS-1,5-3-5.08_1x03_P5.08mm_Horizontal, symbol Connector:Screw_Terminal_01x03
- added C3: 1u, Capacitor_SMD:C_0603_1608Metric, symbol Device:C_Small
- added F1: 0.35A, Fuse:Fuse_1206_3216Metric, symbol Device:Polyfuse_Small
- added J1: USB_C_Receptacle_PowerOnly_6P, Connector_USB:USB_C_Receptacle_HRO_TYPE-C-31-M-17, symbol Connector:USB_C_Receptacle_PowerOnly_6P
- added J4: MAX31865, Connector_PinHeader_2.54mm:PinHeader_1x08_P2.54mm_Vertical, symbol Connector:Conn_01x08_Pin
- added R1: 5.1k, Resistor_SMD:R_0603_1608Metric, symbol Device:R_Small
- added R4, R5: 10k, Resistor_SMD:R_0603_1608Metric, symbol Device:R_Small
- added U1: TPS60403DBV, Package_TO_SOT_SMD:SOT-23-5, symbol Regulator_SwitchedCapacitor:TPS60403DBV
- C2: value 1u -> 2.2u
- J3: renamed from J1; now not fitted; now left out of the parts list
- R2: value 100 -> 5.1k
- U2: now not fitted; now left out of the parts list
- U3: renamed from U1; value (none) -> ESP32_30Pin; now not fitted; now left out of the parts list
- U4: renamed from U3; value TL072 -> TLV9062; footprint Package_DIP:DIP-8_W7.62mm -> Package_SO:TSSOP-8_4.4x3mm_P0.65mm; symbol Amplifier_Operational:TL072 -> Amplifier_Operational:TLV9062
- renumbered J3 to J2, R1 to R3
Connections:
- net +3V3: now also J4.1 (Pin_1), J4.2 (Pin_2)
- net +5V: now also F1.2
- net GND: now also R2.2, C3.2, J1.A12 (GND), J1.B12 (GND), J1.SH (SHIELD), J4.3 (Pin_3), R1.2, U1.4 (GND); no longer C1.1, U4.5 (+)
- net RE: now also R5.1; no longer R3.2
- net VREF: now also R4.1, U1.2 (IN); no longer R2.2
- net MAX31865_RDY: now reaches U3.20 (GPIO4)
- net MAX31865_RDY: now also J4.8 (Pin_8)
- net MAX31865_CS: now reaches U3.23 (GPIO5)
- net MAX31865_CS: now also J4.7 (Pin_7)
- net MAX31865_CLK: now reaches U3.24 (GPIO18)
- net MAX31865_CLK: now also J4.4 (Pin_4)
- net MAX31865_SDO: now reaches U3.25 (GPIO19)
- net MAX31865_SDO: now also J4.5 (Pin_5)
- net MAX31865_SDI: now reaches U3.30 (GPIO23)
- net MAX31865_SDI: now also J4.6 (Pin_6)
- net at J3.7 (Pin_7), R3.1: now also C3.1; no longer C1.2
- net VADC_OUT: now reaches U4.6 (-), U4.7
- net VADC_OUT: now also R3.2
- net -5V renamed -3V3
- net -3V3: now also C2.1, U1.1 (OUT)
- new net: F1.1, J1.A9 (VBUS), J1.B9 (VBUS)
- new net: J1.A5 (CC1), R1.1
- new net: R4.2, R5.2, U4.5 (+)
- new net: C1.2, U1.3 (C_{FLY-})
- new net: C1.1, U1.5 (C_{FLY+})
- new net: J1.B5 (CC2), R2.1
- now unconnected: J3.8 (Pin_8)
- no-connect marks 27 -> 23
Other:
- moved on the sheet: H1, H2, H3, J2, R3, U4A, U4B, U4C

Commit message: Updated PCB
Parts:
- J2: value Screw_Terminal_01x02 -> Aviation_6Pin_GX16; footprint TerminalBlock_Phoenix:TerminalBlock_Phoenix_MKDS-1,5-2-5.08_1x02_P5.08mm_Horizontal -> TerminalBlock_Phoenix:TerminalBlock_Phoenix_MKDS-1,5-6-5.08_1x06_P5.08mm_Horizontal; symbol Connector:Screw_Terminal_01x02 -> Connector:Screw_Terminal_01x06
- R1, R2: footprint Resistor_SMD:R_0603_1608Metric -> Resistor_SMD:R_0402_1005Metric
Connections:
- net V- renamed WE
- no-connect marks 23 -> 27
Changed lines of the file:
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@@
 	)
 	(no_connect
+		(at 176.53 151.13)
+	)
+	(no_connect
 		(at 107.95 86.36)
 	)
 	(no_connect
+		(at 176.53 146.05)
+	)
+	(no_connect
 		(at 107.95 81.28)
 	)
@@
 	)
 	(no_connect
+		(at 176.53 153.67)
+	)
+	(no_connect
 		(at 135.89 81.28)
 	)
@@
 	)
 	(no_connect
+		(at 176.53 148.59)
+	)
+	(no_connect
 		(at 107.95 63.5)
 	)
@@
 	(wire
 		(pts
-			(xy 184.15 144.78) (xy 177.8 144.78)
+			(xy 182.88 140.97) (xy 176.53 140.97)
 		)
 		(stroke
@@
 		)
 	)
-	(label "V-"
+	(label "WE"
 		(at 196.85 140.97 180)
 		(effects
@@
 		)
 	)
-	(label "V-"
-		(at 177.8 147.32 0)
+	(label "WE"
+		(at 176.53 143.51 0)
 		(effects
 			(font
@@
 	(symbol
 		(lib_id "power:GND")
-		(at 184.15 144.78 0)
+		(at 182.88 140.97 0)
 		(unit 1)
 		(body_style 1)
@@
 		(fields_autoplaced yes)
 		(property "Reference" "#PWR013"
-			(at 184.15 151.13 0)
+			(at 182.88 147.32 0)
 			(hide yes)
 			(show_name no)
@@
 		)
 		(property "Value" "GND"
-			(at 186.69 146.0499 0)
+			(at 182.88 146.05 0)
 			(show_name no)
 			(do_not_autoplace no)
@@
 					(size 1.27 1.27)
 				)
-				(justify left)
 			)
 		)
 		(property "Footprint" ""
-			(at 184.15 144.78 0)
+			(at 182.88 140.97 0)
 			(hide yes)
 			(show_name no)
@@
 		)
 		(property "Datasheet" ""
-			(at 184.15 144.78 0)
+			(at 182.88 140.97 0)
 			(hide yes)
 			(show_name no)
@@
 		)
 		(property "Description" "Power symbol creates a global label with name \"GND\" , ground"
-			(at 184.15 144.78 0)
+			(at 182.88 140.97 0)
 			(hide yes)
 			(show_name no)
@@
 	)
 	(symbol
-		(lib_id "Connector:Screw_Terminal_01x02")
-		(at 172.72 144.78 0)
+		(lib_id "Connector:Screw_Terminal_01x06")
+		(at 171.45 146.05 0)
 		(mirror y)
 		(unit 1)
@@
 		(in_pos_files yes)
 		(dnp no)
-		(fields_autoplaced yes)
 		(property "Reference" "J2"
-			(at 172.72 138.43 0)
+			(at 171.45 134.62 0)
 			(show_name no)
 			(do_not_autoplace no)
@@
 			)
 		)
-		(property "Value" "Screw_Terminal_01x02"
-			(at 172.72 140.97 0)
+		(property "Value" "Aviation_6Pin_GX16"
+			(at 171.45 137.16 0)
 			(show_name no)
 			(do_not_autoplace no)
@@
 			)
 		)
-		(property "Footprint" "TerminalBlock_Phoenix:TerminalBlock_Phoenix_MKDS-1,5-2-5.08_1x02_P5.08mm_Horizontal"
-			(at 172.72 144.78 0)
+		(property "Footprint" "TerminalBlock_Phoenix:TerminalBlock_Phoenix_MKDS-1,5-6-5.08_1x06_P5.08mm_Horizontal"
+			(at 171.45 146.05 0)
 			(hide yes)
 			(show_name no)
@@
 		)
 		(property "Datasheet" ""
-			(at 172.72 144.78 0)
+			(at 171.45 146.05 0)
 			(hide yes)
 			(show_name no)
@@
 			)
 		)
-		(property "Description" "Generic screw terminal, single row, 01x02, script generated (kicad-library-utils/schlib/autogen/connector/)"
-			(at 172.72 144.78 0)
+		(property "Description" "Generic screw terminal, single row, 01x06, script generated (kicad-library-utils/schlib/autogen/connector/)"
+			(at 171.45 146.05 0)
 			(hide yes)
 			(show_name no)
@@
 		(pin "2"
 		)
+		(pin "3"
+		)
+		(pin "4"
+		)
+		(pin "5"
+		)
+		(pin "6"
+		)
 		(instances
 			(project "ocp"
@@
 			)
 		)
-		(property "Footprint" "Resistor_SMD:R_0603_1608Metric"
+		(property "Footprint" "Resistor_SMD:R_0402_1005Metric"
 			(at 53.34 43.18 0)
 			(hide yes)
@@
 			)
 		)
-		(property "Footprint" "Resistor_SMD:R_0603_1608Metric"
+		(property "Footprint" "Resistor_SMD:R_0402_1005Metric"
 			(at 53.34 45.72 0)
 			(hide yes)

Commit message: Updated PCB
Parts:
- removed F1: 0.35A, Fuse:Fuse_1206_3216Metric, symbol Device:Polyfuse_Small
- removed J1: USB_C_Receptacle_PowerOnly_6P, Connector_USB:USB_C_Receptacle_HRO_TYPE-C-31-M-17, symbol Connector:USB_C_Receptacle_PowerOnly_6P
- removed R1, R2: 5.1k, Resistor_SMD:R_0402_1005Metric, symbol Device:R_Small
- added H4: MountingHole, MountingHole:MountingHole_2.7mm_M2.5, symbol Mechanical:MountingHole
- added J5: UART, Connector_PinHeader_2.54mm:PinHeader_1x04_P2.54mm_Vertical, symbol Connector:Conn_01x04_Pin
- C1, C3: footprint Capacitor_SMD:C_0603_1608Metric -> Capacitor_SMD:C_0402_1005Metric
Connections:
- net +3V3: now also J5.1 (Pin_1); no longer J4.2 (Pin_2)
- net GND: now also J4.2 (Pin_2), J5.4 (Pin_4); no longer J4.3 (Pin_3)
- net RX: now reaches U3.27 (GPIO3)
- net RX: now also J5.3 (Pin_3)
- net TX: now reaches U3.28 (GPIO1)
- net TX: now also J5.2 (Pin_2)
- no-connect marks 27 -> 26
Other:
- added sheet USBC (USBC.kicad_sch)
- company: (none) -> Indriya Sensotech Private Limited
- title: (none) -> OCP Meter
- moved on the sheet: C1, C2, C3, H1, H2, H3, J3, J4, R3, U1, U2, U3

Commit message: Updated PCB
Parts:
- added C4: 1u, Capacitor_SMD:C_0402_1005Metric, symbol Device:C_Small
- R4, R5: value 10k -> 10k 0.1%
Connections:
- net GND: now also C4.2
- net VREF: now also C4.1
Other:
- moved on the sheet: R5, U4A
Changed lines of the file:
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@@
 	(wire
 		(pts
-			(xy 196.85 149.86) (xy 196.85 146.05)
+			(xy 193.04 149.86) (xy 193.04 146.05)
+		)
+		(stroke
+			(width 0)
+			(type default)
+		)
+	)
+	(wire
+		(pts
+			(xy 24.13 119.38) (xy 34.29 119.38)
 		)
 		(stroke
@@
 	(wire
 		(pts
-			(xy 212.09 149.86) (xy 212.09 143.51)
+			(xy 208.28 149.86) (xy 208.28 143.51)
 		)
 		(stroke
@@
 	(wire
 		(pts
+			(xy 24.13 109.22) (xy 24.13 119.38)
+		)
+		(stroke
+			(width 0)
+			(type default)
+		)
+	)
+	(wire
+		(pts
 			(xy 246.38 44.45) (xy 240.03 44.45)
 		)
@@
 	(wire
 		(pts
-			(xy 196.85 149.86) (xy 212.09 149.86)
+			(xy 193.04 149.86) (xy 208.28 149.86)
 		)
 		(stroke
@@
 	)
 	(label "WE"
-		(at 196.85 140.97 180)
+		(at 193.04 140.97 180)
 		(effects
 			(font
@@
 	)
 	(label "RE"
-		(at 212.09 143.51 0)
+		(at 208.28 143.51 0)
 		(effects
 			(font
@@
 	)
 	(symbol
+		(lib_id "Device:C_Small")
+		(at 24.13 106.68 0)
+		(mirror y)
+		(unit 1)
+		(body_style 1)
+		(exclude_from_sim no)
+		(in_bom yes)
+		(on_board yes)
+		(in_pos_files yes)
+		(dnp no)
+		(property "Reference" "C4"
+			(at 21.59 105.4162 0)
+			(show_name no)
+			(do_not_autoplace no)
+			(effects
+				(font
+					(size 1.27 1.27)
+				)
+				(justify left)
+			)
+		)
+		(property "Value" "1u"
+			(at 21.59 107.9562 0)
+			(show_name no)
+			(do_not_autoplace no)
+			(effects
+				(font
+					(size 1.27 1.27)
+				)
+				(justify left)
+			)
+		)
+		(property "Footprint" "Capacitor_SMD:C_0402_1005Metric"
+			(at 24.13 106.68 0)
+			(hide yes)
+			(show_name no)
+			(do_not_autoplace no)
+			(effects
+				(font
+					(size 1.27 1.27)
+				)
+			)
+		)
+		(property "Datasheet" ""
+			(at 24.13 106.68 0)
+			(hide yes)
+			(show_name no)
+			(do_not_autoplace no)
+			(effects
+				(font
+					(size 1.27 1.27)
+				)
+			)
+		)
+		(property "Description" ""
+			(at 24.13 106.68 0)
+			(show_name no)
+			(do_not_autoplace no)
+			(effects
+				(font
+					(size 1.27 1.27)
+				)
+			)
+		)
+		(pin "1"
+		)
+		(pin "2"
+		)
+		(instances
+			(project "ocp"
+				(path "/e6e8fc66-ad6c-42eb-8ba4-37b895f6ea98"
+					(reference "C4")
+					(unit 1)
+				)
+			)
+		)
+	)
+	(symbol
 		(lib_id "power:+3V3")
 		(at 153.67 86.36 0)
@@
 	(symbol
 		(lib_id "Device:R_Small")
-		(at 224.79 143.51 180)
+		(at 224.79 143.51 0)
+		(mirror x)
 		(unit 1)
 		(body_style 1)
@@
 		(dnp no)
 		(property "Reference" "R5"
-			(at 221.234 142.494 0)
+			(at 222.25 142.2399 0)
 			(show_name no)
 			(do_not_autoplace no)
@@
 			)
 		)
-		(property "Value" "10k"
-			(at 224.79 145.288 90)
+		(property "Value" "10k 0.1%"
+			(at 222.25 144.7799 0)
 			(show_name no)
 			(do_not_autoplace no)
@@
 		(lib_id "Device:R_Small")
 		(at 224.79 138.43 0)
+		(mirror y)
 		(unit 1)
 		(body_style 1)
@@
 		(dnp no)
 		(property "Reference" "R4"
-			(at 221.234 136.906 0)
+			(at 222.25 137.1599 0)
 			(show_name no)
 			(do_not_autoplace no)
@@
 			)
 		)
-		(property "Value" "10k"
-			(at 224.79 140.208 90)
+		(property "Value" "10k 0.1%"
+			(at 222.25 139.6999 0)
 			(show_name no)
 			(do_not_autoplace no)
@@
 	(symbol
 		(lib_id "Amplifier_Operational:TLV9062")
-		(at 204.47 143.51 0)
+		(at 200.66 143.51 0)
 		(unit 1)
 		(body_style 1)
@@
 		(fields_autoplaced yes)
 		(property "Reference" "U4"
-			(at 204.47 133.35 0)
+			(at 200.66 133.35 0)
 			(show_name no)
 			(do_not_autoplace no)
@@
 		)
 		(property "Value" "TLV9062"
-			(at 204.47 135.89 0)
+			(at 200.66 135.89 0)
 			(show_name no)
 			(do_not_autoplace no)
@@
 		)
 		(property "Footprint" "Package_SO:TSSOP-8_4.4x3mm_P0.65mm"
-			(at 204.47 143.51 0)
+			(at 200.66 143.51 0)
 			(hide yes)
 			(show_name no)
@@
 		)
 		(property "Datasheet" "https://www.ti.com/lit/ds/symlink/tlv9062.pdf"
-			(at 204.47 143.51 0)
+			(at 200.66 143.51 0)
 			(hide yes)
 			(show_name no)
@@
 		)
 		(property "Description" "Dual Operational Amplifiers, SOIC-8/TSSOP-8/VSSOP-8"
-			(at 204.47 143.51 0)
+			(at 200.66 143.51 0)
 			(hide yes)
 			(show_name no)
